File: daemon_full_body_tracker.kicad_sch (KiCad schematic)
At the start: 48 parts, among them IC1 nPM1100-CAAA-E-R7, IC2 NRF52805-CAAA-B-R7, J1 150mAh, J3 P70-5100045, J5 P70-5100045, U1 BMM350, U2 BHI360, Y1 ECS-.327-9-34QN-TR, Y2 ECS-320-8-37B2-CTN-TR

Commit message: added todo list for next revision
Other:
- note added: "TODO: have a 0ohm resistor and pin to power nRF52805 with different voltage for programming with DK"

Commit message: updated todo list
Other:
- note added: "TODO: add 0ohm resistor and pin to power nRF52805 with different voltage for programming with DK add 2x TXB0101DBVR 1-channel voltage translators for SWDIO and SWDCLK"
- note removed: "TODO: have a 0ohm resistor and pin to power nRF52805 with different voltage for programming with DK"
Changed lines of the file:
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@@
     (effects (font (size 2.54 2.54) bold (color 72 72 72 1)) (justify left bottom))
   )
-  (text "TODO:\nhave a 0ohm resistor and pin to power nRF52805 with different voltage for programming with DK"
+  (text "TODO:\nadd 0ohm resistor and pin to power nRF52805 with different voltage for programming with DK\nadd 2x TXB0101DBVR 1-channel voltage translators for SWDIO and SWDCLK"
     (at 19.685 20.955 0)
     (effects (font (size 1.27 1.27)) (justify left bottom))

Commit message: updated todo list
Other:
- note added: "TODO: - add 0ohm resistor in series with VDD to nrf52805 - add pin to power nRF52805 with different voltage for programming with DK - add 2x TXB0101DBVR 1-channel voltage translators for SWDIO and SWDCLK"
- note removed: "TODO: add 0ohm resistor and pin to power nRF52805 with different voltage for programming with DK add 2x TXB0101DBVR 1-channel voltage translators for SWDIO and SWDCLK"
Changed lines of the file:
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@@
     (effects (font (size 2.54 2.54) bold (color 72 72 72 1)) (justify left bottom))
   )
-  (text "TODO:\nadd 0ohm resistor and pin to power nRF52805 with different voltage for programming with DK\nadd 2x TXB0101DBVR 1-channel voltage translators for SWDIO and SWDCLK"
-    (at 19.685 20.955 0)
+  (text "TODO:\n- add 0ohm resistor in series with VDD to nrf52805\n- add pin to power nRF52805 with different voltage for programming with DK\n- add 2x TXB0101DBVR 1-channel voltage translators for SWDIO and SWDCLK"
+    (at 19.685 25.4 0)
     (effects (font (size 1.27 1.27)) (justify left bottom))
   )
